Commit message: added meshes and small change

File: pal_gripper_description/urdf/gripper.urdf.xacro (robot description, xacro)
@@ -2,5 +2,5 @@
 <robot xmlns:xacro="http://ros.org/wiki/xacro">
   <!--File includes-->
-  <xacro:include filename="$(find pal_urdf_utils)/urdf/deg_to_rad.urdf.xacro" />
+  <xacro:include filename="$(find pal_urdf_utils)/urdf/deg_to_rad.xacro" />
   <xacro:include filename="$(find pal_gripper_description)/urdf/gripper.gazebo.xacro" />
   <xacro:property name="gripper_eps" value="0.001" />
@@ -77,5 +77,5 @@
     <material>Gazebo/Black</material>
   </gazebo>
-  <joint name="${name}_right_finger_joint" type="prismatic">
+  <joint name="${name}_right_finger_joint" type="fixed">
     <origin rpy="0 0 0" xyz="0. 0 0" />
     <parent link="${name}_link" />
@@ -115,5 +115,5 @@
     <material>Gazebo/Black</material>
   </gazebo>
-  <joint name="${name}_left_finger_joint" type="prismatic">
+  <joint name="${name}_left_finger_joint" type="fixed">
     <origin rpy="0 0 0" xyz="0. 0 0" />
     <parent link="${name}_link" />
